File: Battery/Battery.sch (KiCad schematic (older format))
At the start: 3 parts

Commit message: 4mdOtraDalja
Parts:
- 9V1: footprint Battery_Holder:SMTU2032 -> Battery_Holder:1072 Battery Holder
Changed lines of the file:
@@
 F 0 "9V1" H 3967 3985 50  0000 C CNN
 F 1 "SMTU2032" H 3967 4076 50  0000 C CNN
-F 2 "Battery_Holder:SMTU2032" H 4050 4100 50  0001 C CNN
+F 2 "Battery_Holder:1072 Battery Holder" H 4050 4100 50  0001 C CNN
 F 3 "" H 4050 4100 50  0001 C CNN
 	1    4050 4100
